Commit message: Fixed vikram's motion

File: urdf/vikram_igvc.urdf (robot description, URDF)
Before this commit: robot vikram, 6 links, 5 joints
Links:
- link castor_ball: mass 1 -> 3
- link castor_cylinder: mass 1 -> 2
- link wheel1: mass 2 -> 5; geometry collision cylinder length=0.073987 radius=0.2; visual mesh filename=package://vikram_sim/meshes/igvc/wheel.dae
- link wheel2: mass 2 -> 5; geometry collision cylinder length=0.073987 radius=0.2; visual mesh filename=package://vikram_sim/meshes/igvc/wheel.dae
- link zed_camera: mass 1 -> 0.5
Joints:
- joint body_to_castor_cylinder: origin xyz=0.62 -0.008 -0.15 rpy=0 0 0 -> xyz=0.62 -0.008 -0.15 rpy=0 0.112383 0
- joint body_to_wheel1: origin xyz=-0.019369 -0.32336 0 rpy=0 0 1.5707 -> xyz=-0.019369 -0.35 0 rpy=0 0 1.5707
- joint cylinder_to_castor_ball: origin xyz=0 0 -0.065 rpy=0 0 0 -> xyz=0 0 -0.065 rpy=0 0.132544 0

Commit message: Perfected odom and cmd_vel plots

File: urdf/vikram_igvc.urdf (robot description, URDF)
Before this commit: robot vikram, 6 links, 5 joints
Joints:
- joint body_to_castor_cylinder: origin xyz=0.62 -0.008 -0.15 rpy=0 0.112383 0 -> xyz=-0.609078 -0.008 -0.1 rpy=0 -0.012285 0
- joint body_to_wheel1: axis -1 0 0 -> 1 0 0
- joint body_to_wheel2: axis 1 0 0 -> -1 0 0; origin xyz=-0.019369 0.32336 0 rpy=0 0 -1.5707 -> xyz=-0.019369 0.4 0 rpy=0 0 -1.5707
- joint camera_to_body: origin xyz=0.20 -0.015 0.705 rpy=0 0 3.14 -> xyz=-0.15 0.025 0.705 rpy=0 0 0

Commit message: added pointcloud things

File: urdf/vikram_igvc.urdf (robot description, URDF)
Before this commit: robot vikram, 6 links, 5 joints
Links:
- added link perpendicular, mass 0; collision box size=0.0001 0.00001 0.00001; visual box size=0.0001 0.00001 0.00001
Joints:
- added joint perp: type fixed, parent base_link, child perpendicular, origin xyz=0.15 0 1.58 rpy=-1.5707 0 0

Commit message: changed somethings

File: urdf/vikram_igvc.urdf (robot description, URDF)
Before this commit: robot vikram, 7 links, 6 joints
Joints:
- joint perp: origin xyz=0.15 0 1.58 rpy=-1.5707 0 0 -> xyz=0.15 0 1.58 rpy=-1.5707 0 -1.5707

Commit message: Added plugins for GPS

File: urdf/vikram_igvc.urdf (robot description, URDF)
Before this commit: robot vikram, 7 links, 6 joints
Links:
- added link gps_link, mass 1; collision box size=0.1 0.1 0.1; visual box size=0.1 0.1 0.1
Joints:
- added joint gps_joint: type fixed, parent base_link, child gps_link
